Commit message: Update robot_core.xacro

File: description/robot_core.xacro (robot description, xacro)
@@ -1,69 +1,115 @@
 <?xml version="1.0"?>
 <robot xmlns:xacro="http://www.ros.org/wiki/xacro">
-    <material name="blue">
-        <color rgba="0.2 0.2 1 1"/>
-    </material>
-    <material name="black">
-        <color rgba="0 0 0 1"/>
-    </material>
+    <!-- Base Link (Reference Frame) -->
     <link name="base_link">
+        <!-- No geometry or visual as it serves as a reference frame -->
+    </link>
+    <!-- Back Body Link -->
+    <link name="back_body">
         <visual>
-            <origin xyz="0 0 0.0305" rpy="0 0 0" />
+            <geometry>
+                <box size="0.18 0.18 0.09"/>
+            </geometry>
+            <material name="black">
+                <color rgba="0 0 0 1"/>
+            </material>
         </visual>
     </link>
-    <link name="chasis_back">
+    <!-- Joint between base_link and back_body -->
+    <joint name="back_body_joint" type="fixed">
+        <parent link="base_link"/>
+        <child link="back_body"/>
+        <origin xyz="0 0 0.045" rpy="0 0 0"/>
+    </joint>
+    <!-- Front Body Link -->
+    <link name="front_body">
         <visual>
-        <origin xyz="0 0 0" rpy="0 0 0" />
-        <geometry>
-            <box size="0.18 0.18 0.09" />
-        </geometry>
-        <material name="black"/>
-        </visual>
-        <collision>
-            <origin xyz="0 0 0" rpy="0 0 0" />
             <geometry>
-                <box size="0.18 0.18 0.09" />
+                <box size="0.18 0.18 0.09"/>
             </geometry>
-        </collision>
-        <inertial>
-            <origin xyz="0 0 0" rpy="0 0 0" />
-            <mass value="1" />
-            <inertia ixx="0.16666666666666666" ixy="0" ixz="0" iyy="0.16666666666666666" iyz="0" izz="0.16666666666666666" />
-        </inertial>
-    </link>
-    <joint name="base_link_to_chasis_back" type="fixed">
-        <parent link="base_link" />
-        <child link="chasis_back" />
-        <origin xyz="0.03 0 0.045" rpy="0 0 0" />
-    </joint>
-    <link name="left_wheel_back">
-        <visual>
-            <origin xyz="0 0 0" rpy="0 0 0" />
-            <geometry>
-                <cylinder radius="0.0305" length="0.025" />
-            </geometry>
-            <material name="blue"/>
+            <material name="black">
+                <color rgba="0 0 0 1"/>
+            </material>
         </visual>
     </link>
-    <joint name="chasis_back_to_left_wheel_back" type="continuous">
-        <parent link="base_link" />
-        <child link="left_wheel_back" />
-        <origin xyz="0 0.08 0" rpy="${pi/2} 0 0" />
+    <!-- Center Joint (between front and back sections) -->
+    <joint name="center_joint" type="revolute">
+        <parent link="back_body"/>
+        <child link="front_body"/>
+        <origin xyz="0 0 0.045" rpy="0 0 0"/>
         <axis xyz="0 0 1"/>
+        <limit lower="-1.5708" upper="1.5708" effort="10" velocity="1"/>
     </joint>
-    <link name="right_wheel_back">
+    <!-- Front Left Wheel Link and Joint -->
+    <link name="front_left_wheel">
         <visual>
-            <origin xyz="0 0 0" rpy="0 0 0" />
             <geometry>
-                <cylinder radius="0.0305" length="0.025" />
+                <cylinder radius="0.0305" length="0.025"/>
             </geometry>
-            <material name="blue"/>
+            <material name="yellow">
+                <color rgba="1 1 0 1"/>
+            </material>
         </visual>
     </link>
-    <joint name="chasis_back_to_right_wheel_back" type="continuous">
-        <parent link="base_link" />
-        <child link="right_wheel_back" />
-        <origin xyz="0 -0.08 0" rpy="-${pi/2} 0 0" />
-        <axis xyz="0 0 1"/>
+    <joint name="front_left_wheel_joint" type="revolute">
+        <parent link="front_body"/>
+        <child link="front_left_wheel"/>
+        <origin xyz="0.09 0.09 0" rpy="0 1.5708 0"/>
+        <axis xyz="0 1 0"/>
+        <limit lower="0" upper="0" effort="5" velocity="10"/>
+    </joint>
+    <!-- Front Right Wheel Link and Joint -->
+    <link name="front_right_wheel">
+        <visual>
+            <geometry>
+                <cylinder radius="0.0305" length="0.025"/>
+            </geometry>
+            <material name="yellow">
+                <color rgba="1 1 0 1"/>
+            </material>
+        </visual>
+    </link>
+    <joint name="front_right_wheel_joint" type="revolute">
+        <parent link="front_body"/>
+        <child link="front_right_wheel"/>
+        <origin xyz="0.09 -0.09 0" rpy="0 1.5708 0"/>
+        <axis xyz="0 1 0"/>
+        <limit lower="0" upper="0" effort="5" velocity="10"/>
+    </joint>
+    <!-- Back Left Wheel Link and Joint -->
+    <link name="back_left_wheel">
+        <visual>
+            <geometry>
+                <cylinder radius="0.0305" length="0.025"/>
+            </geometry>
+            <material name="yellow">
+                <color rgba="1 1 0 1"/>
+            </material>
+        </visual>
+    </link>
+    <joint name="back_left_wheel_joint" type="revolute">
+        <parent link="back_body"/>
+        <child link="back_left_wheel"/>
+        <origin xyz="-0.09 0.09 0" rpy="0 1.5708 0"/>
+        <axis xyz="0 1 0"/>
+        <limit lower="0" upper="0" effort="5" velocity="10"/>
+    </joint>
+    <!-- Back Right Wheel Link and Joint -->
+    <link name="back_right_wheel">
+        <visual>
+            <geometry>
+                <cylinder radius="0.0305" length="0.025"/>
+            </geometry>
+            <material name="yellow">
+                <color rgba="1 1 0 1"/>
+            </material>
+        </visual>
+    </link>
+    <joint name="back_right_wheel_joint" type="revolute">
+        <parent link="back_body"/>
+        <child link="back_right_wheel"/>
+        <origin xyz="-0.09 -0.09 0" rpy="0 1.5708 0"/>
+        <axis xyz="0 1 0"/>
+        <limit lower="0" upper="0" effort="5" velocity="10"/>
     </joint>
 </robot>

Commit message: Update robot_core.xacro

File: description/robot_core.xacro (robot description, xacro)
@@ -1,5 +1,5 @@
 <?xml version="1.0"?>
 <robot xmlns:xacro="http://www.ros.org/wiki/xacro">
-    <!-- Base Link (Reference Frame) -->
+      <!-- Base Link (Reference Frame) -->
     <link name="base_link">
         <!-- No geometry or visual as it serves as a reference frame -->
@@ -16,5 +16,5 @@
         </visual>
     </link>
-    <!-- Joint between base_link and back_body -->
+    <!-- Fixed Joint between base_link and back_body -->
     <joint name="back_body_joint" type="fixed">
         <parent link="base_link"/>
@@ -33,9 +33,9 @@
         </visual>
     </link>
-    <!-- Center Joint (between front and back sections) -->
+    <!-- Center Joint (between back_body and front_body) -->
     <joint name="center_joint" type="revolute">
         <parent link="back_body"/>
         <child link="front_body"/>
-        <origin xyz="0 0 0.045" rpy="0 0 0"/>
+        <origin xyz="0.09 0 0.045" rpy="0 0 0"/>
         <axis xyz="0 0 1"/>
         <limit lower="-1.5708" upper="1.5708" effort="10" velocity="1"/>
@@ -52,10 +52,9 @@
         </visual>
     </link>
-    <joint name="front_left_wheel_joint" type="revolute">
+    <joint name="front_left_wheel_joint" type="continuous">
         <parent link="front_body"/>
         <child link="front_left_wheel"/>
-        <origin xyz="0.09 0.09 0" rpy="0 1.5708 0"/>
+        <origin xyz="0.09 0.09 -0.045" rpy="0 1.5708 0"/>
         <axis xyz="0 1 0"/>
-        <limit lower="0" upper="0" effort="5" velocity="10"/>
     </joint>
     <!-- Front Right Wheel Link and Joint -->
@@ -70,10 +69,9 @@
         </visual>
     </link>
-    <joint name="front_right_wheel_joint" type="revolute">
+    <joint name="front_right_wheel_joint" type="continuous">
         <parent link="front_body"/>
         <child link="front_right_wheel"/>
-        <origin xyz="0.09 -0.09 0" rpy="0 1.5708 0"/>
+        <origin xyz="0.09 -0.09 -0.045" rpy="0 1.5708 0"/>
         <axis xyz="0 1 0"/>
-        <limit lower="0" upper="0" effort="5" velocity="10"/>
     </joint>
     <!-- Back Left Wheel Link and Joint -->
@@ -88,10 +86,9 @@
         </visual>
     </link>
-    <joint name="back_left_wheel_joint" type="revolute">
+    <joint name="back_left_wheel_joint" type="continuous">
         <parent link="back_body"/>
         <child link="back_left_wheel"/>
-        <origin xyz="-0.09 0.09 0" rpy="0 1.5708 0"/>
+        <origin xyz="-0.09 0.09 -0.045" rpy="0 1.5708 0"/>
         <axis xyz="0 1 0"/>
-        <limit lower="0" upper="0" effort="5" velocity="10"/>
     </joint>
     <!-- Back Right Wheel Link and Joint -->
@@ -106,10 +103,9 @@
         </visual>
     </link>
-    <joint name="back_right_wheel_joint" type="revolute">
+    <joint name="back_right_wheel_joint" type="continuous">
         <parent link="back_body"/>
         <child link="back_right_wheel"/>
-        <origin xyz="-0.09 -0.09 0" rpy="0 1.5708 0"/>
+        <origin xyz="-0.09 -0.09 -0.045" rpy="0 1.5708 0"/>
         <axis xyz="0 1 0"/>
-        <limit lower="0" upper="0" effort="5" velocity="10"/>
     </joint>
 </robot>

Commit message: Update URDF

File: description/robot_core.xacro (robot description, xacro)
@@ -1,9 +1,11 @@
 <?xml version="1.0"?>
 <robot xmlns:xacro="http://www.ros.org/wiki/xacro">
-      <!-- Base Link (Reference Frame) -->
     <link name="base_link">
-        <!-- No geometry or visual as it serves as a reference frame -->
     </link>
-    <!-- Back Body Link -->
+    <joint name="back_body_joint" type="fixed">
+        <parent link="base_link"/>
+        <child link="back_body"/>
+        <origin xyz="0 0 0.045" rpy="0 0 0"/>
+    </joint>
     <link name="back_body">
         <visual>
@@ -16,13 +18,14 @@
         </visual>
     </link>
-    <!-- Fixed Joint between base_link and back_body -->
-    <joint name="back_body_joint" type="fixed">
-        <parent link="base_link"/>
-        <child link="back_body"/>
-        <origin xyz="0 0 0.045" rpy="0 0 0"/>
+    <joint name="center_joint" type="revolute">
+        <parent link="back_body"/>
+        <child link="front_body"/>
+        <origin xyz="0.09 0 0" rpy="0 0 0"/>
+        <axis xyz="0 0 1"/>
+        <limit lower="-1.5708" upper="1.5708" effort="10" velocity="1"/>
     </joint>
-    <!-- Front Body Link -->
     <link name="front_body">
         <visual>
+            <origin xyz="0.09 0 0"/>
             <geometry>
                 <box size="0.18 0.18 0.09"/>
@@ -33,13 +36,43 @@
         </visual>
     </link>
-    <!-- Center Joint (between back_body and front_body) -->
-    <joint name="center_joint" type="revolute">
-        <parent link="back_body"/>
-        <child link="front_body"/>
-        <origin xyz="0.09 0 0.045" rpy="0 0 0"/>
+    <link name="back_left_wheel">
+        <visual>
+            <geometry>
+                <cylinder radius="0.0305" length="0.025"/>
+            </geometry>
+            <material name="yellow">
+                <color rgba="1 1 0 1"/>
+            </material>
+        </visual>
+    </link>
+    <joint name="back_left_wheel_joint" type="continuous">
+        <parent link="base_link"/>
+        <child link="back_left_wheel"/>
+        <origin xyz="0 0.09 0" rpy="-${pi/2} 0 0"/>
+        <axis xyz="0 0 -1"/>
+    </joint>
+    <link name="back_right_wheel">
+        <visual>
+            <geometry>
+                <cylinder radius="0.0305" length="0.025"/>
+            </geometry>
+            <material name="yellow">
+                <color rgba="1 1 0 1"/>
+            </material>
+        </visual>
+    </link>
+    <joint name="back_right_wheel_joint" type="continuous">
+        <parent link="base_link"/>
+        <child link="back_right_wheel"/>
+        <origin xyz="0 -0.09 0" rpy="${pi/2} 0 0"/>
         <axis xyz="0 0 1"/>
-        <limit lower="-1.5708" upper="1.5708" effort="10" velocity="1"/>
     </joint>
-    <!-- Front Left Wheel Link and Joint -->
+    <link name="base_front">
+    </link>
+    <joint name="base_front_joint" type="fixed">
+        <parent link="front_body"/>
+        <child link="base_front"/>
+        <origin xyz="0.09 0 -0.045" rpy="0 0 0"/>
+    </joint>
     <link name="front_left_wheel">
         <visual>
@@ -53,10 +86,9 @@
     </link>
     <joint name="front_left_wheel_joint" type="continuous">
-        <parent link="front_body"/>
+        <parent link="base_front"/>
         <child link="front_left_wheel"/>
-        <origin xyz="0.09 0.09 -0.045" rpy="0 1.5708 0"/>
-        <axis xyz="0 1 0"/>
+        <origin xyz="0 0.09 0" rpy="-${pi/2} 0 0"/>
+        <axis xyz="0 0 -1"/>
     </joint>
-    <!-- Front Right Wheel Link and Joint -->
     <link name="front_right_wheel">
         <visual>
@@ -70,42 +102,8 @@
     </link>
     <joint name="front_right_wheel_joint" type="continuous">
-        <parent link="front_body"/>
+        <parent link="base_front"/>
         <child link="front_right_wheel"/>
-        <origin xyz="0.09 -0.09 -0.045" rpy="0 1.5708 0"/>
-        <axis xyz="0 1 0"/>
-    </joint>
-    <!-- Back Left Wheel Link and Joint -->
-    <link name="back_left_wheel">
-        <visual>
-            <geometry>
-                <cylinder radius="0.0305" length="0.025"/>
-            </geometry>
-            <material name="yellow">
-                <color rgba="1 1 0 1"/>
-            </material>
-        </visual>
-    </link>
-    <joint name="back_left_wheel_joint" type="continuous">
-        <parent link="back_body"/>
-        <child link="back_left_wheel"/>
-        <origin xyz="-0.09 0.09 -0.045" rpy="0 1.5708 0"/>
-        <axis xyz="0 1 0"/>
-    </joint>
-    <!-- Back Right Wheel Link and Joint -->
-    <link name="back_right_wheel">
-        <visual>
-            <geometry>
-                <cylinder radius="0.0305" length="0.025"/>
-            </geometry>
-            <material name="yellow">
-                <color rgba="1 1 0 1"/>
-            </material>
-        </visual>
-    </link>
-    <joint name="back_right_wheel_joint" type="continuous">
-        <parent link="back_body"/>
-        <child link="back_right_wheel"/>
-        <origin xyz="-0.09 -0.09 -0.045" rpy="0 1.5708 0"/>
-        <axis xyz="0 1 0"/>
+        <origin xyz="0 -0.09 0" rpy="${pi/2} 0 0"/>
+        <axis xyz="0 0 1"/>
     </joint>
 </robot>

Commit message: Add colission and inertia to URDF

File: description/robot_core.xacro (robot description, xacro)
@@ -1,4 +1,5 @@
 <?xml version="1.0"?>
 <robot xmlns:xacro="http://www.ros.org/wiki/xacro">
+    <xacro:include filename="inertial_macros.xacro" />
     <link name="base_link">
     </link>
@@ -17,4 +18,12 @@
             </material>
         </visual>
+        <collision>
+            <geometry>
+                <box size="0.18 0.18 0.09"/>
+            </geometry>
+        </collision>
+        <xacro:inertial_box mass="1" x="0.18" y="0.18" z="0.09">
+            <origin xyz="0 0 0" rpy="0 0 0"/>
+        </xacro:inertial_box>
     </link>
     <joint name="center_joint" type="revolute">
@@ -35,4 +44,13 @@
             </material>
         </visual>
+        <collision>
+            <origin xyz="0.09 0 0"/>
+            <geometry>
+                <box size="0.18 0.18 0.09"/>
+            </geometry>
+        </collision>
+        <xacro:inertial_box mass="1" x="0.18" y="0.18" z="0.09">
+            <origin xyz="0.09 0 0" rpy="0 0 0"/>
+        </xacro:inertial_box>
     </link>
     <link name="back_left_wheel">
@@ -45,4 +63,12 @@
             </material>
         </visual>
+        <collision>
+            <geometry>
+                <cylinder radius="0.0305" length="0.025"/>
+            </geometry>
+        </collision>
+        <xacro:inertial_cylinder mass="0.05" length="0.0025" radius="0.0305">
+            <origin xyz="0 0 0" rpy="0 0 0"/>
+        </xacro:inertial_cylinder>
     </link>
     <joint name="back_left_wheel_joint" type="continuous">
@@ -61,4 +87,12 @@
             </material>
         </visual>
+        <collision>
+            <geometry>
+                <cylinder radius="0.0305" length="0.025"/>
+            </geometry>
+        </collision>
+        <xacro:inertial_cylinder mass="0.05" length="0.0025" radius="0.0305">
+            <origin xyz="0 0 0" rpy="0 0 0"/>
+        </xacro:inertial_cylinder>
     </link>
     <joint name="back_right_wheel_joint" type="continuous">
@@ -84,4 +118,12 @@
             </material>
         </visual>
+        <collision>
+            <geometry>
+                <cylinder radius="0.0305" length="0.025"/>
+            </geometry>
+        </collision>
+        <xacro:inertial_cylinder mass="0.05" length="0.0025" radius="0.0305">
+            <origin xyz="0 0 0" rpy="0 0 0"/>
+        </xacro:inertial_cylinder>
     </link>
     <joint name="front_left_wheel_joint" type="continuous">
@@ -100,4 +142,12 @@
             </material>
         </visual>
+        <collision>
+            <geometry>
+                <cylinder radius="0.0305" length="0.025"/>
+            </geometry>
+        </collision>
+        <xacro:inertial_cylinder mass="0.05" length="0.0025" radius="0.0305">
+            <origin xyz="0 0 0" rpy="0 0 0"/>
+        </xacro:inertial_cylinder>
     </link>
     <joint name="front_right_wheel_joint" type="continuous">

Commit message: update robot model

File: description/robot_core.xacro (robot description, xacro)
@@ -75,5 +75,5 @@
         <parent link="base_link"/>
         <child link="back_left_wheel"/>
-        <origin xyz="0 0.09 0" rpy="-${pi/2} 0 0"/>
+        <origin xyz="0 0.1025 0" rpy="-${pi/2} 0 0"/>
         <axis xyz="0 0 -1"/>
     </joint>
@@ -99,13 +99,6 @@
         <parent link="base_link"/>
         <child link="back_right_wheel"/>
-        <origin xyz="0 -0.09 0" rpy="${pi/2} 0 0"/>
+        <origin xyz="0 -0.1025 0" rpy="${pi/2} 0 0"/>
         <axis xyz="0 0 1"/>
-    </joint>
-    <link name="base_front">
-    </link>
-    <joint name="base_front_joint" type="fixed">
-        <parent link="front_body"/>
-        <child link="base_front"/>
-        <origin xyz="0.09 0 -0.045" rpy="0 0 0"/>
     </joint>
     <link name="front_left_wheel">
@@ -128,7 +121,7 @@
     </link>
     <joint name="front_left_wheel_joint" type="continuous">
-        <parent link="base_front"/>
+        <parent link="front_body"/>
         <child link="front_left_wheel"/>
-        <origin xyz="0 0.09 0" rpy="-${pi/2} 0 0"/>
+        <origin xyz="0.09 0.1025 -0.045" rpy="-${pi/2} 0 0"/>
         <axis xyz="0 0 -1"/>
     </joint>
@@ -152,7 +145,7 @@
     </link>
     <joint name="front_right_wheel_joint" type="continuous">
-        <parent link="base_front"/>
+        <parent link="front_body"/>
         <child link="front_right_wheel"/>
-        <origin xyz="0 -0.09 0" rpy="${pi/2} 0 0"/>
+        <origin xyz="0.09 -0.1025 -0.045" rpy="${pi/2} 0 0"/>
         <axis xyz="0 0 1"/>
     </joint>
