Commit message: update xacro

File: description/robot.urdf.xacro (robot description, xacro)
@@ -2,3 +2,5 @@
 <robot xmlns:xacro="http://www.ros.org/wiki/xacro"  name="artibot">
     <xacro:include filename="robot_core.xacro" />
+    <!-- <xacro:include filename="gazebo_control.xacro" /> -->
+    <xacro:include filename="lidar.xacro" />
 </robot>

File: description/robot_core.xacro (robot description, xacro)
@@ -4,10 +4,10 @@
     <link name="base_link">
     </link>
-    <joint name="back_body_joint" type="fixed">
+    <joint name="front_body_joint" type="fixed">
         <parent link="base_link"/>
-        <child link="back_body"/>
-        <origin xyz="0 0 0.045" rpy="0 0 0"/>
+        <child link="front_body"/>
+        <origin xyz="-0.027 0 0.045" rpy="0 0 0"/>
     </joint>
-    <link name="back_body">
+    <link name="front_body">
         <visual>
             <geometry>
@@ -27,79 +27,7 @@
         </xacro:inertial_box>
     </link>
-    <joint name="center_joint" type="revolute">
-        <parent link="back_body"/>
-        <child link="front_body"/>
-        <origin xyz="0.09 0 0" rpy="0 0 0"/>
-        <axis xyz="0 0 1"/>
-        <limit lower="-1.5708" upper="1.5708" effort="10" velocity="1"/>
-    </joint>
-    <link name="front_body">
-        <visual>
-            <origin xyz="0.09 0 0"/>
-            <geometry>
-                <box size="0.18 0.18 0.09"/>
-            </geometry>
-            <material name="black">
-                <color rgba="0 0 0 1"/>
-            </material>
-        </visual>
-        <collision>
-            <origin xyz="0.09 0 0"/>
-            <geometry>
-                <box size="0.18 0.18 0.09"/>
-            </geometry>
-        </collision>
-        <xacro:inertial_box mass="1" x="0.18" y="0.18" z="0.09">
-            <origin xyz="0.09 0 0" rpy="0 0 0"/>
-        </xacro:inertial_box>
-    </link>
-    <link name="back_left_wheel">
-        <visual>
-            <geometry>
-                <cylinder radius="0.0305" length="0.025"/>
-            </geometry>
-            <material name="yellow">
-                <color rgba="1 1 0 1"/>
-            </material>
-        </visual>
-        <collision>
-            <geometry>
-                <cylinder radius="0.0305" length="0.025"/>
-            </geometry>
-        </collision>
-        <xacro:inertial_cylinder mass="0.05" length="0.0025" radius="0.0305">
-            <origin xyz="0 0 0" rpy="0 0 0"/>
-        </xacro:inertial_cylinder>
-    </link>
-    <joint name="back_left_wheel_joint" type="continuous">
-        <parent link="base_link"/>
-        <child link="back_left_wheel"/>
-        <origin xyz="0 0.1025 0" rpy="-${pi/2} 0 0"/>
-        <axis xyz="0 0 -1"/>
-    </joint>
-    <link name="back_right_wheel">
-        <visual>
-            <geometry>
-                <cylinder radius="0.0305" length="0.025"/>
-            </geometry>
-            <material name="yellow">
-                <color rgba="1 1 0 1"/>
-            </material>
-        </visual>
-        <collision>
-            <geometry>
-                <cylinder radius="0.0305" length="0.025"/>
-            </geometry>
-        </collision>
-        <xacro:inertial_cylinder mass="0.05" length="0.0025" radius="0.0305">
-            <origin xyz="0 0 0" rpy="0 0 0"/>
-        </xacro:inertial_cylinder>
-    </link>
-    <joint name="back_right_wheel_joint" type="continuous">
-        <parent link="base_link"/>
-        <child link="back_right_wheel"/>
-        <origin xyz="0 -0.1025 0" rpy="${pi/2} 0 0"/>
-        <axis xyz="0 0 1"/>
-    </joint>
+    <gazebo reference="front_body">
+        <material>Gazebo/Black</material>
+    </gazebo>
     <link name="front_left_wheel">
         <visual>
@@ -120,9 +48,12 @@
         </xacro:inertial_cylinder>
     </link>
-    <joint name="front_left_wheel_joint" type="continuous">
-        <parent link="front_body"/>
+    <gazebo reference="front_left_wheel">
+        <material>Gazebo/Blue</material>
+    </gazebo>
+    <joint name="front_left_wheel_joint" type="fixed">
+        <parent link="base_link"/>
         <child link="front_left_wheel"/>
-        <origin xyz="0.09 0.1025 -0.045" rpy="-${pi/2} 0 0"/>
-        <axis xyz="0 0 -1"/>
+        <origin xyz="0 0.0775 0" rpy="${-pi/2} 0 0"/>
+        <axis xyz="0 0 1"/>
     </joint>
     <link name="front_right_wheel">
@@ -144,9 +75,39 @@
         </xacro:inertial_cylinder>
     </link>
-    <joint name="front_right_wheel_joint" type="continuous">
-        <parent link="front_body"/>
+    <gazebo reference="front_right_wheel">
+        <material>Gazebo/Blue</material>
+    </gazebo>
+    <joint name="front_right_wheel_joint" type="fixed">
+        <parent link="base_link"/>
         <child link="front_right_wheel"/>
-        <origin xyz="0.09 -0.1025 -0.045" rpy="${pi/2} 0 0"/>
+        <origin xyz="0 -0.0775 0" rpy="${-pi/2} 0 0"/>
         <axis xyz="0 0 1"/>
     </joint>
+    <!-- CASTER WHEEL -->
+    <joint name="caster_wheel_joint" type="fixed">
+        <parent link="front_body"/>
+        <child link="caster_wheel"/>
+        <origin xyz="-0.0595 0 -0.045" rpy="0 0 0"/>
+    </joint>
+    <link name="caster_wheel">
+        <visual>
+            <geometry>
+                <sphere radius="0.0305" />
+            </geometry>
+            <material name="black"/>
+        </visual>
+        <collision>
+            <geometry>
+                <sphere radius="0.0305" />
+            </geometry>
+        </collision>
+        <xacro:inertial_sphere mass="0.1" radius="0.0305">
+            <origin xyz="0 0 0" rpy="0 0 0"/>
+        </xacro:inertial_sphere>
+    </link>
+    <gazebo reference="caster_wheel">
+        <material>Gazebo/White</material>
+            <mu1 value="0.001"/>
+            <mu2 value="0.001"/>
+    </gazebo>
 </robot>
