Commit message: update lidar urdf

File: description/lidar.xacro (robot description, xacro)
@@ -5,5 +5,5 @@
         <parent link="front_body"/>
         <child link="laser_frame"/>
-        <origin xyz="0 0 0.056" rpy="0 0 0"/>
+        <origin xyz="0 0 0.056" rpy="0 0 ${pi}"/>
     </joint>
     <link name="laser_frame">
